File: Schematics/Insoleuse/Insoleuse.sch (KiCad schematic (older format))
At the start: 9 parts

Commit message: Update schematics
Parts:
- C1, C2: renamed from C47µf; value C -> 47µf
- R1: renamed from R10K; value R -> 10K
- U?: value NHD-0420H1Z -> LCD 20x4
Connections:
- wire segments 44 -> 52
Other:
- note added: "LCD Module"
- note added: "Power Supply"
- moved on the sheet: U?
